File: hardware/ignition-coil-spark-generator.sch (KiCad schematic (older format))
At the start: 20 parts

Commit message: Better component names in schematic
Parts:
- D?: value LED -> LED_INDICATOR
- D?: value LED -> LED_SPARK_0
- D?: value LED -> LED_SPARK_1
- E?: value SPARK_GAP -> SPARK_0
- E?: value SPARK_GAP -> SPARK_1
- P?: value CONN_01X02 -> LOGIC_12V
- P?: value CONN_01X02 -> SPARK_12V
- SW?: value SW_PUSH -> RESET
Changed lines of the file:
@@
 P 1050 3400
 F 0 "P?" H 1050 3550 50  0000 C CNN
-F 1 "CONN_01X02" V 1150 3400 50  0000 C CNN
+F 1 "LOGIC_12V" V 1150 3400 50  0000 C CNN
 F 2 "" H 1050 3400 50  0000 C CNN
 F 3 "" H 1050 3400 50  0000 C CNN
@@
 P 4000 4100
 F 0 "D?" H 4000 4200 50  0000 C CNN
-F 1 "LED" H 4000 4000 50  0000 C CNN
+F 1 "LED_INDICATOR" H 4000 4000 50  0000 C CNN
 F 2 "" H 4000 4100 50  0000 C CNN
 F 3 "" H 4000 4100 50  0000 C CNN
@@
 P 5450 2550
 F 0 "E?" H 5450 2630 50  0000 C CNN
-F 1 "SPARK_GAP" H 5450 2475 50  0000 C CNN
+F 1 "SPARK_0" H 5450 2475 50  0000 C CNN
 F 2 "" H 5450 2480 50  0001 C CNN
 F 3 "" V 5450 2550 50  0001 C CNN
@@
 P 5950 2550
 F 0 "E?" H 5950 2630 50  0000 C CNN
-F 1 "SPARK_GAP" H 5950 2475 50  0000 C CNN
+F 1 "SPARK_1" H 5950 2475 50  0000 C CNN
 F 2 "" H 5950 2480 50  0001 C CNN
 F 3 "" V 5950 2550 50  0001 C CNN
@@
 P 5000 4600
 F 0 "D?" H 5000 4700 50  0000 C CNN
-F 1 "LED" H 5000 4500 50  0000 C CNN
+F 1 "LED_SPARK_0" H 5000 4500 50  0000 C CNN
 F 2 "" H 5000 4600 50  0000 C CNN
 F 3 "" H 5000 4600 50  0000 C CNN
@@
 P 6200 4600
 F 0 "D?" H 6200 4700 50  0000 C CNN
-F 1 "LED" H 6200 4500 50  0000 C CNN
+F 1 "LED_SPARK_1" H 6200 4500 50  0000 C CNN
 F 2 "" H 6200 4600 50  0000 C CNN
 F 3 "" H 6200 4600 50  0000 C CNN
@@
 P 3700 4900
 F 0 "SW?" H 3850 5010 50  0000 C CNN
-F 1 "SW_PUSH" H 3700 4820 50  0000 C CNN
+F 1 "RESET" H 3700 4820 50  0000 C CNN
 F 2 "" H 3700 4900 50  0000 C CNN
 F 3 "" H 3700 4900 50  0000 C CNN
@@
 P 1050 2700
 F 0 "P?" H 1050 2850 50  0000 C CNN
-F 1 "CONN_01X02" V 1150 2700 50  0000 C CNN
+F 1 "SPARK_12V" V 1150 2700 50  0000 C CNN
 F 2 "" H 1050 2700 50  0000 C CNN
 F 3 "" H 1050 2700 50  0000 C CNN

Commit message: Add spark power indicator led
Parts:
- added D?: LED, symbol LED
- added R?: R, symbol R
Connections:
- net +12V: now also D?.2 (A)
- net GNDPWR: now also R?.2
- new net: D?.1 (K), R?.1
Changed lines of the file:
@@
 $EndComp
 Wire Wire Line
-	4500 3000 4500 4600
+	4500 3000 4500 3900
+Wire Wire Line
+	4500 3900 4500 4600
 Connection ~ 4500 3900
 $Comp
@@
 $EndComp
 Wire Wire Line
-	5700 4950 5700 3900
+	5700 4950 5700 4600
+Wire Wire Line
+	5700 4600 5700 3900
 Connection ~ 5700 4600
 $Comp
@@
 $EndComp
 Wire Wire Line
-	1250 2650 1550 2650
+	1250 2650 1350 2650
 $Comp
 L GNDPWR #PWR?
 U 1 1 5954555D
-P 1250 2750
-F 0 "#PWR?" H 1250 2550 50  0001 C CNN
-F 1 "GNDPWR" H 1250 2620 50  0000 C CNN
-F 2 "" H 1250 2700 50  0000 C CNN
-F 3 "" H 1250 2700 50  0000 C CNN
-	1    1250 2750
+P 1250 2900
+F 0 "#PWR?" H 1250 2700 50  0001 C CNN
+F 1 "GNDPWR" H 1250 2770 50  0000 C CNN
+F 2 "" H 1250 2850 50  0000 C CNN
+F 3 "" H 1250 2850 50  0000 C CNN
+	1    1250 2900
 	1    0    0    -1
 $EndComp
@@
 L +12V #PWR?
 U 1 1 59545599
-P 1550 2650
-F 0 "#PWR?" H 1550 2500 50  0001 C CNN
-F 1 "+12V" H 1550 2790 50  0000 C CNN
-F 2 "" H 1550 2650 50  0000 C CNN
-F 3 "" H 1550 2650 50  0000 C CNN
-	1    1550 2650
+P 1250 2650
+F 0 "#PWR?" H 1250 2500 50  0001 C CNN
+F 1 "+12V" H 1250 2790 50  0000 C CNN
+F 2 "" H 1250 2650 50  0000 C CNN
+F 3 "" H 1250 2650 50  0000 C CNN
+	1    1250 2650
 	1    0    0    -1
 $EndComp
 NoConn ~ 2150 3600
 NoConn ~ 2150 3500
+$Comp
+L LED D?
+U 1 1 595519F1
+P 1550 2650
+F 0 "D?" H 1550 2750 50  0000 C CNN
+F 1 "LED" H 1550 2550 50  0000 C CNN
+F 2 "" H 1550 2650 50  0000 C CNN
+F 3 "" H 1550 2650 50  0000 C CNN
+	1    1550 2650
+	-1   0    0    1
+$EndComp
+$Comp
+L R R?
+U 1 1 59551A58
+P 1600 2900
+F 0 "R?" V 1680 2900 50  0000 C CNN
+F 1 "R" V 1600 2900 50  0000 C CNN
+F 2 "" V 1530 2900 50  0000 C CNN
+F 3 "" H 1600 2900 50  0000 C CNN
+	1    1600 2900
+	0    1    1    0
+$EndComp
+Wire Wire Line
+	1750 2650 1750 2900
+Wire Wire Line
+	1450 2900 1250 2900
+Wire Wire Line
+	1250 2900 1250 2750
 $EndSCHEMATC

Commit message: Connect ground and power ground together - otherwise fets act strange and heat up a lot
Connections:
- net GNDPWR is gone; now on net GND: D?.2 (A), D?.2 (A), P?.1 (P1), Q?.3 (S), Q?.3 (S), R?.2
Changed lines of the file:
@@
 	4350 3700 4350 4950
 Wire Wire Line
-	4350 4950 5700 4950
+	5700 4950 4350 4950
 Wire Wire Line
 	2150 4100 2050 4100
@@
 $EndComp
 Wire Wire Line
-	4500 3000 4500 3900
-Wire Wire Line
-	4500 3900 4500 4600
+	4500 3000 4500 4600
 Connection ~ 4500 3900
 $Comp
@@
 $EndComp
 Wire Wire Line
-	5700 4950 5700 4600
-Wire Wire Line
-	5700 4600 5700 3900
+	5700 3900 5700 4950
 Connection ~ 5700 4600
 $Comp
@@
 Wire Wire Line
 	1250 2900 1250 2750
+$Comp
+L GND #PWR?
+U 1 1 5958027A
+P 1100 3900
+F 0 "#PWR?" H 1100 3650 50  0001 C CNN
+F 1 "GND" H 1100 3750 50  0000 C CNN
+F 2 "" H 1100 3900 50  0000 C CNN
+F 3 "" H 1100 3900 50  0000 C CNN
+	1    1100 3900
+	1    0    0    -1
+$EndComp
+$Comp
+L GNDPWR #PWR?
+U 1 1 595802BA
+P 1450 3900
+F 0 "#PWR?" H 1450 3700 50  0001 C CNN
+F 1 "GNDPWR" H 1450 3770 50  0000 C CNN
+F 2 "" H 1450 3850 50  0000 C CNN
+F 3 "" H 1450 3850 50  0000 C CNN
+	1    1450 3900
+	1    0    0    -1
+$EndComp
+Wire Wire Line
+	1100 3900 1450 3900
 $EndSCHEMATC
